File: pcb/WM8978.kicad_sch (KiCad schematic)
At the start: 50 parts, among them CN2 HEADPHONE 3.5mm, SW4 RESET, U15 AMS1117-3.3, U16 WM8978GEFL/RV, U17 STM32F407VET6, X3 8MHz CL=12pF

Commit message: Refactor schematic into functional hierarchy
Split USB power, STM32, WM8978, and audio outputs into separate sheets; correct power decoupling and regulator specification; document the reviewed signal chain; remove the obsolete firmware tree.
Parts:
- removed C60, C67, C70, C71, C72, C73, C74, C75, C76, C94: 100nF, Capacitor_SMD:C_0603_1608Metric, symbol WM8978-easyedapro:CapAcitance
- removed C64: 1uF, Capacitor_SMD:C_0603_1608Metric, symbol WM8978-easyedapro:CapAcitance
- removed C65, C66: 2.2uF, Capacitor_SMD:C_0603_1608Metric, symbol WM8978-easyedapro:CapAcitance
- removed C68, C69: 18pF, Capacitor_SMD:C_0603_1608Metric, symbol WM8978-easyedapro:CapAcitance
- removed C77, C78: 10uF, Capacitor_SMD:C_0805_2012Metric, symbol WM8978-easyedapro:CapAcitance
- removed C83: 4.7uF, Capacitor_SMD:C_0603_1608Metric, symbol WM8978-easyedapro:CL21A106KPFNNNF
- removed C86, C87: 220uF/6.3V, Capacitor_SMD:CP_Elec_6.3x5.8, symbol WM8978-easyedapro:220UF/16V_C9900022878
- removed C88, C90, C92: 100nF, Capacitor_SMD:C_0603_1608Metric, symbol WM8978-easyedapro:CL03A104KO3NNNC
- removed C89, C91, C93: 10uF, Capacitor_SMD:C_0805_2012Metric, symbol WM8978-easyedapro:CL21A106KPFNNNF
- removed C95: 4.7uF, Capacitor_SMD:C_0805_2012Metric, symbol WM8978-easyedapro:CapAcitance
- removed CN2: HEADPHONE 3.5mm, WM8978-import-fps:AUDIO-TH_PJ-3136-B, symbol WM8978-easyedapro:PJ-3136-B
- removed D1, D2: PESD5V0U1BA, Diode_SMD:D_SOD-323, symbol Device:D_TVS
- removed H10: SWD 1x4, Connector_PinHeader_2.54mm:PinHeader_1x04_P2.54mm_Vertical, symbol WM8978-easyedapro:PZ254V-11-04P_C2691448
- removed R50, R56: 10k, Resistor_SMD:R_0603_1608Metric, symbol WM8978-easyedapro:电阻
- removed R51, R52: 0R, Resistor_SMD:R_0603_1608Metric, symbol WM8978-easyedapro:电阻
- removed R53, R54: 22R, Resistor_SMD:R_0603_1608Metric, symbol WM8978-easyedapro:电阻
- removed R57: 1M, Resistor_SMD:R_0603_1608Metric, symbol WM8978-easyedapro:电阻
- removed R62: 10k, Resistor_SMD:R_0603_1608Metric, symbol WM8978-easyedapro:FRC0603F1002TS
- removed R63, R64: 4.7k, Resistor_SMD:R_0603_1608Metric, symbol WM8978-easyedapro:RC0603JR-074K7L
- removed R65, R66: 5.1k, Resistor_SMD:R_0603_1608Metric, symbol WM8978-easyedapro:0603WAF5101T5E
- removed SPK2: SPEAKER 8R BTL, Connector_JST:JST_PH_B2B-PH-K_1x02_P2.00mm_Vertical, symbol WM8978-easyedapro:FS-2308
- removed SW4: RESET, Button_Switch_SMD:SW_SPST_TL3342, symbol WM8978-easyedapro:轻触按键x2
- removed U15: AMS1117-3.3, Package_TO_SOT_SMD:SOT-223, symbol WM8978-easyedapro:AMS1117
- removed U16: WM8978GEFL/RV, Package_DFN_QFN:QFN-32-1EP_5x5mm_P0.5mm_EP3.1x3.1mm, symbol WM8978-easyedapro:WM8978GEFL/RV
- removed U17: STM32F407VET6, Package_QFP:LQFP-100_14x14mm_P0.5mm, symbol WM8978-easyedapro:STM32F407VET6
- removed USB2: USB-C USB2 DEVICE, WM8978-import-fps:USB_TYPE-C-16P, symbol WM8978-easyedapro:USB_TYPE-C-16P
- removed X3: 8MHz CL=12pF, Crystal:Crystal_SMD_5032-2Pin_5.0x3.2mm, symbol WM8978-easyedapro:9C0803LCSC-DDK2S
Connections:
- no-connect marks 89 -> 0
Other:
- added sheet Headphone and Speaker Outputs (04_audio_output.kicad_sch)
- added sheet STM32F407 Core, Clock and Debug (02_stm32.kicad_sch)
- added sheet USB Type-C and Power (01_usb_power.kicad_sch)
- added sheet WM8978 Codec (03_wm8978.kicad_sch)
- note removed: "3.3V POWER"
- note removed: "ADC/MIC/LSE/EEPROM/EXTERNAL AMP REMOVED"
- note removed: "C86/C87: 220uF headphone DC-blocking capacitors; use common 6.3x5.8mm SMD electrolytic"
- note removed: "R53/R54 place close to MCU USB pins"
- note removed: "RESET"
- note removed: "SPK2: WM8978 BTL output - do not connect either speaker wire to GND"
- note removed: "STM32F407 + 8MHz HSE"
- note removed: "SWD"
- note removed: "USB 2.0 DEVICE"
- note removed: "WM8978 USB PLAYBACK"
