File: pcb/WM8978.kicad_sch (KiCad schematic)
At the start: 0 parts

Commit message: 修复原理图电源网络并更新项目文档
Parts:
- added C60, C67, C70, C71, C72, C73, C74, C75, C76, C94: 100nF, Capacitor_SMD:C_0603_1608Metric, symbol WM8978-easyedapro:CapAcitance
- added C64, C79, C80: 1uF, Capacitor_SMD:C_0603_1608Metric, symbol WM8978-easyedapro:CapAcitance
- added C65, C66: 2.2uF, Capacitor_SMD:C_0603_1608Metric, symbol WM8978-easyedapro:CapAcitance
- added C68, C69: 18pF, Capacitor_SMD:C_0603_1608Metric, symbol WM8978-easyedapro:CapAcitance
- added C77, C83, C89, C91, C93, C95, C96: 4.7uF, Capacitor_SMD:C_0603_1608Metric, symbol WM8978-easyedapro:CapAcitance
- added C78: 10uF, Capacitor_SMD:C_0603_1608Metric, symbol WM8978-easyedapro:CapAcitance
- added C86, C87: 220uF/16V, Capacitor_SMD:CP_Elec_6.3x5.8, symbol WM8978-easyedapro:220UF/16V_C9900022878
- added C88, C90, C92: 100nF, Capacitor_SMD:C_0603_1608Metric, symbol WM8978-easyedapro:CL03A104KO3NNNC
- added CN2: HEADPHONE 3.5mm, WM8978-import-fps:AUDIO-TH_PJ-3136-B, symbol WM8978-easyedapro:PJ-3136-B
- added D1, D2: PESD5V0U1BA, Diode_SMD:D_SOD-323, symbol Device:D_TVS
- added H10: SWD 1x4, Connector_PinHeader_2.54mm:PinHeader_1x04_P2.54mm_Vertical, symbol WM8978-easyedapro:PZ254V-11-04P_C2691448
- added MIC1: ELECTRET MIC, WM8978-import-fps:MIC-TH_BD4.0-P1.40-D0.4-L-FD, symbol WM8978-easyedapro:GMI4015P-2C-42DB
- added R50, R69: 10k, Resistor_SMD:R_0603_1608Metric, symbol WM8978-easyedapro:电阻
- added R51, R52: 0R, Resistor_SMD:R_0603_1608Metric, symbol WM8978-easyedapro:电阻
- added R53, R54: 22R, Resistor_SMD:R_0603_1608Metric, symbol WM8978-easyedapro:电阻
- added R62: 10k, Resistor_SMD:R_0603_1608Metric, symbol WM8978-easyedapro:FRC0603F1002TS
- added R63, R64: 4.7k, Resistor_SMD:R_0603_1608Metric, symbol WM8978-easyedapro:RC0603JR-074K7L
- added R65, R66: 5.1k, Resistor_SMD:R_0603_1608Metric, symbol WM8978-easyedapro:0603WAF5101T5E
- added R67: 1k, Resistor_SMD:R_0603_1608Metric, symbol WM8978-easyedapro:电阻
- added R68: 2.2k, Resistor_SMD:R_0603_1608Metric, symbol WM8978-easyedapro:FRC0603F1002TS
- added SPK2: SPEAKER 8R BTL, Connector_JST:JST_PH_B2B-PH-K_1x02_P2.00mm_Vertical, symbol WM8978-easyedapro:FS-2308
- added SW4: RESET, Button_Switch_SMD:SW_SPST_TL3342, symbol WM8978-easyedapro:轻触按键x2
- added SW5: BOOT, Button_Switch_SMD:SW_SPST_TL3342, symbol WM8978-easyedapro:轻触按键x2
- added U15: TLV1117LV33DCYR, Package_TO_SOT_SMD:SOT-223, symbol WM8978-easyedapro:AMS1117
- added U16: WM8978GEFL/RV, Package_DFN_QFN:QFN-32-1EP_5x5mm_P0.5mm_EP3.1x3.1mm, symbol WM8978-easyedapro:WM8978GEFL/RV
- added U17: STM32F407VET6, Package_QFP:LQFP-100_14x14mm_P0.5mm, symbol WM8978-easyedapro:STM32F407VET6
- added USB2: USB-C USB2 DEVICE, WM8978-import-fps:USB_TYPE-C-16P, symbol WM8978-easyedapro:USB_TYPE-C-16P
- added X3: 8MHz CL=12pF, Crystal:Crystal_SMD_5032-2Pin_5.0x3.2mm, symbol WM8978-easyedapro:9C0803LCSC-DDK2S
Connections:
- net 3V3: now also C70.1, C71.1, C72.1, C73.1, C74.1, C76.1, C78.1, C88.1, C90.1, C94.1, C95.1, H10.1, R52.2, R63.2, R64.2, SW5.2, U15.2 (VOUT), U15.4 (TAB), U16.13 (DCVDD), U16.14 (DBVDD), U16.31 (AVDD), U17.100 (VDD), U17.11 (VDD), U17.19 (VDD), U17.28 (VDD), U17.50 (VDD), U17.6 (VBAT), U17.75 (VDD)
- net GND: now also C60.1, C64.1, C65.2, C66.2, C67.1, C68.2, C69.2, C70.2, C71.2, C72.2, C73.2, C74.2, C75.2, C76.2, C77.2, C78.2, C88.2, C90.2, C92.1, C94.2, C95.2, CN2.2, D1.2 (A2), D2.2 (A2), H10.4, MIC1.2, R50.2, R51.2, R62.1, R65.2, R66.2, R69.2, SW4.2, U15.1 (GND), U16.12 (DGND), U16.15 (CSB/GPIO1), U16.24 (SPKGND), U16.28 (AGND), U16.33 (EPAD), U17.10 (VSS), U17.27 (VSS), U17.74 (VSS), U17.99 (VSS), USB2.1 (EP), USB2.2 (EP), USB2.3 (EP), USB2.4 (EP), USB2.A1 (GND), USB2.A12 (GND), USB2.B1 (GND), USB2.B12 (GND)
- net VBUS_5V: now also C75.1, C77.1, C92.2, R67.1, U15.3 (VIN), U16.26 (SPKVDD), USB2.A4 (VBUS), USB2.A9 (VBUS), USB2.B4 (VBUS), USB2.B9 (VBUS)
- new net: R64.1, U16.16 (SCLK)
- new net: C67.2, SW4.1, U17.14 (NRST)
- new net: D2.1 (A1), R54.1, USB2.A7 (DN1), USB2.B7 (DN2)
- new net: C65.1, U17.73 (VCAP_2)
- new net: H10.2, U17.72 (PA13(JTMS-SWDIO))
- new net: H10.3, U17.76 (PA14(JTCK-SWCLK))
- new net: C87.2, CN2.3
- new net: D1.1 (A1), R53.1, USB2.A6 (DP1), USB2.B6 (DP2)
- new net: C68.1, U17.12 (PH0-OSC_IN(PH0)), X3.2 (OSC2)
- new net: R66.1, USB2.B5 (CC2)
- new net: R69.1, U17.37 (PB2-BOOT1(PB2))
- new net: R67.2, U17.68 (PA9)
- new net: C69.1, U17.13 (PH1-OSC_OUT(PH1)), X3.1 (OSC1)
- new net: R51.1, U17.20 (VSSA)
- new net: C66.1, U17.49 (VCAP_1)
- new net: MIC1.1, R68.2
- new net: R50.1, SW5.1, U17.94 (BOOT0)
- new net: R65.1, USB2.A5 (CC1)
- new net: R63.1, U16.17 (SDIN)
- new net: C86.2, CN2.4
- new net CODEC_SCLK: U17.87 (PD6)
- new net CODEC_SDIN: U17.88 (PD7)
- new net HP_L: C86.1, U16.30 (LOUT1)
- new net HP_R: C87.1, U16.29 (ROUT1)
- new net I2S_ADCDAT: U16.9 (ADCDAT), U17.17 (PC2)
- new net I2S_BCLK: U16.8 (BCLK), U17.52 (PB13)
- new net I2S_DACDAT: U16.10 (DACDAT), U17.18 (PC3)
- new net I2S_LRCLK: U16.7 (LRC), U17.51 (PB12)
- new net I2S_MCLK: U16.11 (MCLK), U17.63 (PC6)
- new net MICBIAS: R68.1
- new net MIC_LIN: U16.2 (LIN)
- new net MIC_LIP: U16.1 (LIP)
- new net MODE: R62.2, U16.18 (MODE)
- new net SPK_N: SPK2.2, U16.25 (LOUT2)
- new net SPK_P: SPK2.1, U16.23 (ROUT2)
- new net USB_DM: R54.2, U17.70 (PA11)
- new net USB_DP: R53.2, U17.71 (PA12)
- new net VDDA: C60.2, C64.2, R52.1, U17.21 (VREF+), U17.22 (VDDA)
- no-connect marks 0 -> 77
Other:
- removed sheet Headphone and Speaker Outputs
- removed sheet STM32F407 Core, Clock and Debug
- removed sheet USB Type-C and Power
- removed sheet WM8978 Codec
- note added: "Headphone and Speaker Outputs"
- note added: "STM32F407 Core, USB and SWD"
- note added: "USB Type-C and Power"
- note added: "WM8978 Codec and Microphone Front End"
- company: USB playback reference redesign -> USB full-duplex audio reference
- title: STM32F407 + WM8978 USB Audio -> STM32F407 + WM8978 USB Audio - Single Sheet

Commit message: 更新单页原理图布局并同步 PCB
Connections:
- net 3V3: now also C89.1, C91.1
- net GND: now also C80.2, C83.2, C89.2, C91.2, C93.1, C96.2
- net MIC_LIN: now also C80.1
- net MIC_LIP: now also C79.1
- net VBUS_5V: now also C93.2
- net at C83.1: now also U16.27 (VMID)
- net at C96.1: now also U16.32 (MICBIAS)
- net at MIC1.1, R68.2: now also C79.2
- net HP_L: no longer names the net of U16.30 (LOUT1)
- net HP_L: now also C87.1; no longer C86.1
- net HP_R: no longer names the net of U16.29 (ROUT1)
- net HP_R: now also C86.1; no longer C87.1
- net SPK_N: no longer names the net of SPK2.2, U16.25 (LOUT2)
- net SPK_P: no longer names the net of SPK2.1, U16.23 (ROUT2)
Other:
- note removed: "Headphone and Speaker Outputs"
- moved on the sheet: C75, C76, C77, C78, C79, C80, C83, C86, C87, C88, C89, C90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

Commit message: 9.22
Parts:
- removed C60, C67, C70, C71, C72, C73, C74, C94: 100nF, Capacitor_SMD:C_0603_1608Metric, symbol WM8978-easyedapro:CapAcitance
- removed C64: 1uF, Capacitor_SMD:C_0603_1608Metric, symbol WM8978-easyedapro:CapAcitance
- removed C65, C66: 2.2uF, Capacitor_SMD:C_0603_1608Metric, symbol WM8978-easyedapro:CapAcitance
- removed C68, C69: 18pF, Capacitor_SMD:C_0603_1608Metric, symbol WM8978-easyedapro:CapAcitance
- removed C95: 4.7uF, Capacitor_SMD:C_0603_1608Metric, symbol WM8978-easyedapro:CapAcitance
- removed H10: SWD 1x4, Connector_PinHeader_2.54mm:PinHeader_1x04_P2.54mm_Vertical, symbol WM8978-easyedapro:PZ254V-11-04P_C2691448
- removed R50, R69: 10k, Resistor_SMD:R_0603_1608Metric, symbol WM8978-easyedapro:电阻
- removed R51, R52: 0R, Resistor_SMD:R_0603_1608Metric, symbol WM8978-easyedapro:电阻
- removed R67: 1k, Resistor_SMD:R_0603_1608Metric, symbol WM8978-easyedapro:电阻
- removed SW4: RESET, Button_Switch_SMD:SW_SPST_TL3342, symbol WM8978-easyedapro:轻触按键x2
- removed SW5: BOOT, Button_Switch_SMD:SW_SPST_TL3342, symbol WM8978-easyedapro:轻触按键x2
- removed U17: STM32F407VET6, Package_QFP:LQFP-100_14x14mm_P0.5mm, symbol WM8978-easyedapro:STM32F407VET6
- removed X3: 8MHz CL=12pF, Crystal:Crystal_SMD_5032-2Pin_5.0x3.2mm, symbol WM8978-easyedapro:9C0803LCSC-DDK2S
- added C100, C98: 10uF / 16V, Capacitor_SMD:C_0603_1608Metric, symbol Device:C
- added C101: 1uF / 16V, Capacitor_SMD:C_0603_1608Metric, symbol Device:C
- added C102, C104, C106, C97, C99: 100nF, Capacitor_SMD:C_0603_1608Metric, symbol Device:C
- added C103: 10nF, Capacitor_SMD:C_0603_1608Metric, symbol Device:C
- added C105: 1uF, Capacitor_SMD:C_0603_1608Metric, symbol Device:C
- added C107: 4.7uF, Capacitor_SMD:C_0603_1608Metric, symbol Device:C
- added J2: JLINK SWD, Connector_JST:JST_XH_B4B-XH-A_1x04_P2.50mm_Vertical, symbol PCM_SparkFun-Connector:Conn_01x04_P2.54mm
- added R70: 10k, Resistor_SMD:R_0603_1608Metric, symbol Device:R
- added R71: 1k, Resistor_SMD:R_0603_1608Metric, symbol Device:R
- added R72: 330R, Resistor_SMD:R_0603_1608Metric, symbol Device:R
- added R73, R75, R76: 33R, Resistor_SMD:R_0603_1608Metric, symbol Device:R
- added R74, R79, R80: 100k, Resistor_SMD:R_0603_1608Metric, symbol Device:R
- added R77: 0R, Resistor_SMD:R_0603_1608Metric, symbol Device:R
- added R78: 61.9k, Resistor_SMD:R_0603_1608Metric, symbol Device:R
- added SW1: RESET, Button_Switch_SMD:SW_Tactile_SPST_NO_Straight_CK_PTS636Sx25SMTRLFS, symbol Switch:SW_Push
- added TP1: RESET, TestPoint:TestPoint_Pad_D1.0mm, symbol Connector:TestPoint
- added TP10: SDA, TestPoint:TestPoint_Pad_D1.0mm, symbol Connector:TestPoint
- added TP11: SCL, TestPoint:TestPoint_Pad_D1.0mm, symbol Connector:TestPoint
- added TP12: FAULT, TestPoint:TestPoint_Pad_D1.0mm, symbol Connector:TestPoint
- added TP2: GND, TestPoint:TestPoint_Pad_D1.0mm, symbol Connector:TestPoint
- added TP3: RAW 5V, TestPoint:TestPoint_Pad_D1.0mm, symbol Connector:TestPoint
- added TP4: 5V, TestPoint:TestPoint_Pad_D1.0mm, symbol Connector:TestPoint
- added TP5: 3V3, TestPoint:TestPoint_Pad_D1.0mm, symbol Connector:TestPoint
- added TP6: CORE, TestPoint:TestPoint_Pad_D1.0mm, symbol Connector:TestPoint
- added TP7: MCLK, TestPoint:TestPoint_Pad_D1.0mm, symbol Connector:TestPoint
- added TP8: BCLK, TestPoint:TestPoint_Pad_D1.0mm, symbol Connector:TestPoint
- added TP9: LRCLK, TestPoint:TestPoint_Pad_D1.0mm, symbol Connector:TestPoint
- added U1: ATSAMD21E18A-A, Package_QFP:TQFP-32_7x7mm_P0.8mm, symbol WM8978-local:SAMD21E18A_Wired
- added U17: TPS2553DBVR, Package_TO_SOT_SMD:SOT-23-6, symbol WM8978-local:TPS2553DBV
- added U18: SN74LVC1G125DBVR, Package_TO_SOT_SMD:SOT-23-5, symbol 74xGxx:74LVC1G125
- added Y1: 12MHz / 3.3V / 50ppm, Oscillator:Oscillator_SMD_Abracon_ASE-4Pin_3.2x2.5mm, symbol Oscillator:ASE-xxxMHz
- C75, C76, C77, C78, C79, C80, C83, C89, C91, C93, C96: symbol WM8978-easyedapro:CapAcitance -> Device:C; Dielectric (none) -> X7R; Voltage (none) -> 16V
- C86, C87: value 220uF/16V -> 470uF/16V; footprint Capacitor_SMD:CP_Elec_6.3x5.8 -> Capacitor_SMD:CP_Elec_8x10.5; symbol WM8978-easyedapro:220UF/16V_C9900022878 -> Device:C_Polarized; Case (none) -> 8mm diameter, 10.2mm nominal height, FK size F; MPN (none) -> EEEFK1C471P; Manufacturer (none) -> Panasonic
- C88, C90, C92: symbol WM8978-easyedapro:CL03A104KO3NNNC -> Device:C; Dielectric (none) -> X7R; Voltage (none) -> 16V
- CN2: MPN (none) -> PJ-3136-B; Manufacturer (none) -> XKB
- R53, R54: symbol WM8978-easyedapro:电阻 -> Device:R
- R62, R68: symbol WM8978-easyedapro:FRC0603F1002TS -> Device:R
- R63, R64: symbol WM8978-easyedapro:RC0603JR-074K7L -> Device:R
- R65, R66: symbol WM8978-easyedapro:0603WAF5101T5E -> Device:R
- U15: MPN (none) -> TLV1117LV33DCYR; Manufacturer (none) -> Texas Instruments
- U16: value WM8978GEFL/RV -> WM8978CGEFL/RV; footprint Package_DFN_QFN:QFN-32-1EP_5x5mm_P0.5mm_EP3.1x3.1mm -> Package_DFN_QFN:QFN-32-1EP_5x5mm_P0.5mm_EP3.45x3.45mm; symbol WM8978-easyedapro:WM8978GEFL/RV -> WM8978-local:WM8978C_Wired; MPN (none) -> WM8978CGEFL/RV; Manufacturer (none) -> Cirrus Logic / Wolfson
- USB2: footprint WM8978-import-fps:USB_TYPE-C-16P -> WM8978-import-fps:USB_C_GCT_USB4105_GF_A; symbol WM8978-easyedapro:USB_TYPE-C-16P -> WM8978-local:USB4105_Wired; MPN (none) -> USB4105-GF-A; Manufacturer (none) -> GCT
Connections:
- net GND: now also C100.2, C101.2, C102.2, C103.2, C104.2, C105.2, C106.2, C107.2, C97.2, C98.2, C99.2, J2.4 (Pin_4), R74.2, R78.2, R79.2, SW1.2, TP2.1, U1.10 (GND), U1.28 (GND), U17.2 (GND), U18.1, U18.3 (GND), Y1.2 (GND)
- net I2S_ADCDAT: now also U1.11 (PA08_/_I2S_RX)
- net I2S_BCLK: now also R75.2, TP8.1, U1.13 (PA10_/_SCK0); no longer U16.8 (BCLK)
- net I2S_DACDAT: now also U1.8 (PA07_/_I2S_TX)
- net I2S_LRCLK: now also R76.2, TP9.1, U1.14 (PA11_/_FS0); no longer U16.7 (LRC)
- net I2S_MCLK: now also R73.2, TP7.1, U1.15 (PA14_/_XIN)
- net MICBIAS: now also C96.1, U16.32 (MICBIAS)
- net USB_DM: now also U1.23 (PA24_/_USB_DM)
- net USB_DP: now also U1.24 (PA25_/_USB_DP)
- net VBUS_5V: now also TP4.1, U17.6 (OUT); no longer USB2.A4 (VBUS), USB2.A9 (VBUS), USB2.B4 (VBUS), USB2.B9 (VBUS)
- net CODEC_SCL: now reaches R64.1, U16.16 (SCLK)
- net CODEC_SCL: now also TP11.1, U1.22 (PA23_/_SCL)
- net CODEC_SDA: now reaches R63.1, U16.17 (SDIN)
- net CODEC_SDA: now also TP10.1, U1.21 (PA22_/_SDA)
- net 3V3 renamed +3V3
- net +3V3: now also C100.1, C103.1, C104.1, C97.1, C98.1, C99.1, J2.1 (Pin_1), R70.1, R71.1, R77.1, R80.1, TP5.1, U1.30 (VDDIN), U1.9 (VDDANA), U18.5 (VCC), Y1.4 (Vdd); no longer U16.31 (AVDD)
- new net: R80.2, TP12.1, U17.4 (~{FAULT})
- new net: R72.2, SW1.1
- new net: R78.1, U17.5 (ILIM)
- new net AUDIO_CLK_EN: R74.1, U1.19 (PA18_/_XO_EN), Y1.1 (EN)
- new net AVDD_3V3: C106.1, C107.1, R77.2, U16.31 (AVDD)
- new net CODEC_BCLK: R75.1, U16.8 (BCLK)
- new net CODEC_LRCLK: R76.1, U16.7 (LRC)
- new net MCLK_BUF: R73.1, U18.4
- new net MCLK_XO: R79.1, U18.2, Y1.3 (OUT)
- new net MCU_RESET_N: C102.1, R70.2, R72.1, TP1.1, U1.26 (~{RESET})
- new net SWCLK: J2.3 (Pin_3), R71.2, U1.31 (PA30_/_SWCLK)
- new net SWDIO: J2.2 (Pin_2), U1.32 (PA31_/_SWDIO)
- new net VBUS_RAW: C105.1, TP3.1, U17.1 (IN), U17.3 (EN), USB2.A4 (VBUS), USB2.A9 (VBUS), USB2.B4 (VBUS), USB2.B9 (VBUS)
- new net VDDCORE: C101.1, TP6.1, U1.29 (VDDCORE)
- no-connect marks 77 -> 24
Other:
- note added: "Boot OSC8M -> PA18 high -> wait >=2 ms -> select XOSC external clock. Before USB suspend: return MCU to internal clock, then disable Y1. U18 provides MCLK fanout drive; place R73 at its output."
- note added: "C86/C87: Panasonic EEEFK1C471P, 470uF / 16V 8 mm can diameter; positive terminal toward codec. SPK2 is BTL: neither terminal connects to ground."
- note added: "Codec is I2S master: LRCLK = 48 kHz, BCLK = 3.072 MHz 32-bit slots / 16-bit samples; R75/R76 close to codec outputs."
- note added: "Continuous signal wiring; labels are annotations. Power/ground use conventional symbols."
- note added: "Firmware: check SAMD21 silicon revision (C/D/H); apply DS80000760 errata. USB async audio needs feedback + DMA buffering; no firmware supplied. Keep speaker off before USB configuration; total continuous load <=350 mA and within the USB host power budget. Verify suspend current on hardware."
- note added: "J2: 1=VTref, 2=SWDIO, 3=SWCLK, 4=GND Debugger nRESET connects to TP1; TP2 is ground."
- note added: "Layout: C106/C107 at AVDD; R77 = 0R default. Use one continuous ground plane. Keep clock/USB away from microphone input; route HP returns away from MIC."
- note added: "SAMD21E18A + WM8978 | USB full-duplex audio | 48 kHz / 16-bit"
- note added: "USB input: R78 = 61.9k / 1%; current limit about 425 mA C105 = 1uF directly on VBUS; output capacitors after soft start."
- note removed: "STM32F407 Core, USB and SWD"
- note removed: "USB Type-C and Power"
- note removed: "WM8978 Codec and Microphone Front End"
- company: USB full-duplex audio reference -> USB full-duplex audio
- title: STM32F407 + WM8978 USB Audio - Single Sheet -> SAMD21E18A + WM8978 USB Audio
- moved on the sheet: CN2, MIC1, SPK2, U15

Commit message: 更新双时钟音频工程并整理中文原理图与检查资料
Parts:
- removed R62: 10k, Resistor_SMD:R_0603_1608Metric, symbol Device:R
- removed R72: 330R, Resistor_SMD:R_0603_1608Metric, symbol Device:R
- removed R77: 0R, Resistor_SMD:R_0603_1608Metric, symbol Device:R
- removed R79, R80: 100k, Resistor_SMD:R_0603_1608Metric, symbol Device:R
- removed SW1: RESET, Button_Switch_SMD:SW_Tactile_SPST_NO_Straight_CK_PTS636Sx25SMTRLFS, symbol Switch:SW_Push
- removed TP1: RESET, TestPoint:TestPoint_Pad_D1.0mm, symbol Connector:TestPoint
- removed TP10: SDA, TestPoint:TestPoint_Pad_D1.0mm, symbol Connector:TestPoint
- removed TP11: SCL, TestPoint:TestPoint_Pad_D1.0mm, symbol Connector:TestPoint
- removed TP12: FAULT, TestPoint:TestPoint_Pad_D1.0mm, symbol Connector:TestPoint
- removed TP2: GND, TestPoint:TestPoint_Pad_D1.0mm, symbol Connector:TestPoint
- removed TP3: RAW 5V, TestPoint:TestPoint_Pad_D1.0mm, symbol Connector:TestPoint
- removed TP4: 5V, TestPoint:TestPoint_Pad_D1.0mm, symbol Connector:TestPoint
- removed TP5: 3V3, TestPoint:TestPoint_Pad_D1.0mm, symbol Connector:TestPoint
- removed TP6: CORE, TestPoint:TestPoint_Pad_D1.0mm, symbol Connector:TestPoint
- removed TP7: MCLK, TestPoint:TestPoint_Pad_D1.0mm, symbol Connector:TestPoint
- removed TP8: BCLK, TestPoint:TestPoint_Pad_D1.0mm, symbol Connector:TestPoint
- removed TP9: LRCLK, TestPoint:TestPoint_Pad_D1.0mm, symbol Connector:TestPoint
- removed U18: SN74LVC1G125DBVR, Package_TO_SOT_SMD:SOT-23-5, symbol 74xGxx:74LVC1G125
- added Y2: 12.288MHz / 3.3V / 50ppm, Oscillator:Oscillator_SMD_Abracon_ASE-4Pin_3.2x2.5mm, symbol Oscillator:ASE-xxxMHz
- J2: symbol PCM_SparkFun-Connector:Conn_01x04_P2.54mm -> WM8978-local:SWD_4pin
Connections:
- net AVDD_3V3 is gone; now on net +3V3: C106.1, C107.1, U16.31 (AVDD)
- net MODE is gone; now on net GND: U16.18 (MODE)
- net +3V3: now also Y2.4 (Vdd)
- net AUDIO_CLK_EN: now also Y2.1 (EN)
- net GND: now also Y2.2 (GND)
- net at C87.2: now also CN2.4; no longer CN2.3
- net at C86.2: now also CN2.3; no longer CN2.4
- net I2S_MCLK renamed AUDIO_MCLK
- net AUDIO_MCLK: no longer U1.15 (PA14_/_XIN)
- net MCLK_BUF renamed AUDIO_OSC
- net AUDIO_OSC: now also Y2.3 (OUT)
- net MCLK_XO renamed MCU_12M
- net MCU_12M: now also U1.15 (PA14_/_XIN)
- no-connect marks 24 -> 25
Other:
- note added: "C86/C87：松下 EEEFK1C471P，470 µF / 16 V。 罐体直径 8 mm；正极朝向音频编解码器。 SPK2 为 BTL 桥接输出，两端均不可接地。"
- note added: "J2 引脚：1=VTref，2=SWDIO，3=SWCLK，4=GND。 四线 SWD 接口，未引出外部复位；必要时断电重启。"
- note added: "SAMD21E18A + WM8978 | USB 全双工音频 | 48 kHz / 16 位"
- note added: "USB 输入：R78 = 61.9 kΩ / 1%，限流约 425 mA。 C105 = 1 µF，直接接 VBUS；输出电容位于软启动开关之后。"
- note added: "使用 OSC8M 启动 → PA18 拉高 → 等待至少 2 ms → 切换至 12 MHz XOSC 外部时钟。 Y1 为单片机及 USB 提供时钟；Y2 的 12.288 MHz 仅供编解码器，编解码器为 I2S 主机。 USB 与音频时钟异步，需使用反馈及 DMA 缓冲。 挂起前：先静音，将单片机切回内部时钟，再关闭 Y1/Y2。"
- note added: "信号采用连续导线连接，标签仅作标注；电源和地使用常规符号。"
- note added: "固件：核对 SAMD21 硅版本（C/D/H），遵循 DS80000760 勘误。 USB 异步音频需反馈及 DMA 缓冲；本工程未提供固件。 USB 配置完成前关闭扬声器；整机持续电流不超过 350 mA， 并满足 USB 主机供电预算；挂起电流需实板验证。"
- note added: "布局：C106/C107 靠近 AVDD；AVDD 直接接 3.3 V。 使用连续完整的地平面；时钟和 USB 走线远离麦克风输入， 耳机回流路径避开麦克风电路。"
- note added: "编解码器使用 Y2 的 12.288 MHz MCLK，关闭 PLL；SYSCLK=256fs。 R6：CLKSEL=MCLK，MCLKDIV=/1，BCLKDIV=/4，MS=1。 LRCLK 为 48 kHz，BCLK 为 3.072 MHz；32 位时隙 / 16 位采样。 SAMD21 的 I2S 时钟单元 0 设为从机；R75/R76 靠近编解码器输出端。"
- note removed: "Boot OSC8M -> PA18 high -> wait >=2 ms -> select XOSC external clock. Before USB suspend: return MCU to internal clock, then disable Y1. U18 provides MCLK fanout drive; place R73 at its output."
- note removed: "C86/C87: Panasonic EEEFK1C471P, 470uF / 16V 8 mm can diameter; positive terminal toward codec. SPK2 is BTL: neither terminal connects to ground."
- note removed: "Codec is I2S master: LRCLK = 48 kHz, BCLK = 3.072 MHz 32-bit slots / 16-bit samples; R75/R76 close to codec outputs."
- note removed: "Continuous signal wiring; labels are annotations. Power/ground use conventional symbols."
- note removed: "Firmware: check SAMD21 silicon revision (C/D/H); apply DS80000760 errata. USB async audio needs feedback + DMA buffering; no firmware supplied. Keep speaker off before USB configuration; total continuous load <=350 mA and within the USB host power budget. Verify suspend current on hardware."
- note removed: "J2: 1=VTref, 2=SWDIO, 3=SWCLK, 4=GND Debugger nRESET connects to TP1; TP2 is ground."
- note removed: "Layout: C106/C107 at AVDD; R77 = 0R default. Use one continuous ground plane. Keep clock/USB away from microphone input; route HP returns away from MIC."
- note removed: "SAMD21E18A + WM8978 | USB full-duplex audio | 48 kHz / 16-bit"
- note removed: "USB input: R78 = 61.9k / 1%; current limit about 425 mA C105 = 1uF directly on VBUS; output capacitors after soft start."
- moved on the sheet: C75, C77, C96

Commit message: 补齐封装关联并绑定原始 3D 模型
补齐 C97～C100 的符号关联，Y1/Y2 使用 Abracon 原厂 STEP，MIC1 使用立创原库 STEP。
CN2 保留现有五脚封装，仅去除原库 CAD 多余的板下插脚，并保存未经修改的六脚原文件。
保留最新存档中的 C97/C98 位置与铺铜调整，记录 54 个器件的关联、模型及原生 STEP 验证结果。
Parts:
- Y1, Y2: footprint Oscillator:Oscillator_SMD_Abracon_ASE-4Pin_3.2x2.5mm -> WM8978-import-fps:Oscillator_SMD_Abracon_ASE-4Pin_3.2x2.5mm
Changed lines of the file:
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@@
 			)
 		)
-		(property "Footprint" "Oscillator:Oscillator_SMD_Abracon_ASE-4Pin_3.2x2.5mm"
+		(property "Footprint" "WM8978-import-fps:Oscillator_SMD_Abracon_ASE-4Pin_3.2x2.5mm"
 			(at 200.66 248.92 0)
 			(hide yes)
@@
 			)
 		)
-		(property "Footprint" "Oscillator:Oscillator_SMD_Abracon_ASE-4Pin_3.2x2.5mm"
+		(property "Footprint" "WM8978-import-fps:Oscillator_SMD_Abracon_ASE-4Pin_3.2x2.5mm"
 			(at 149.86 248.92 0)
 			(hide yes)
