File: pcb/03_wm8978.kicad_sch (KiCad schematic)
At the start: 11 parts, among them U16 WM8978GEFL/RV

Commit message: 修复原理图电源网络并更新项目文档
Parts:
- added C79, C80: 1uF, Capacitor_SMD:C_0603_1608Metric, symbol WM8978-easyedapro:CapAcitance
- added C96: 4.7uF, Capacitor_SMD:C_0603_1608Metric, symbol WM8978-easyedapro:CapAcitance
- added MIC1: ELECTRET MIC, WM8978-import-fps:MIC-TH_BD4.0-P1.40-D0.4-L-FD, symbol WM8978-easyedapro:GMI4015P-2C-42DB
- added R68: 2.2k, Resistor_SMD:R_0603_1608Metric, symbol WM8978-easyedapro:FRC0603F1002TS
- C83: footprint Capacitor_SMD:C_0805_2012Metric -> Capacitor_SMD:C_0603_1608Metric; symbol WM8978-easyedapro:CL21A106KPFNNNF -> WM8978-easyedapro:CapAcitance
- C89, C93: value 10uF -> 4.7uF; footprint Capacitor_SMD:C_0805_2012Metric -> Capacitor_SMD:C_0603_1608Metric; symbol WM8978-easyedapro:CL21A106KPFNNNF -> WM8978-easyedapro:CapAcitance
- C91: value 100nF -> 4.7uF; symbol WM8978-easyedapro:CL21A106KPFNNNF -> WM8978-easyedapro:CapAcitance
Connections:
- net 3V3: no longer C89.2, C91.2
- net GND: now also MIC1.2; no longer C83.1, C89.1, C91.1, C93.1
- net VBUS_5V: no longer C93.2
- net MIC_LIP: now reaches U16.1 (LIP)
- net MIC_LIN: now reaches U16.2 (LIN)
- net MICBIAS: now reaches U16.32 (MICBIAS)
- net MICBIAS: now also R68.1
- net I2S_ADCDAT: now reaches U16.9 (ADCDAT)
- net VMID: no longer names the net of U16.27 (VMID)
- net VMID: no longer C83.2
- new net: MIC1.1, R68.2
- no-connect marks 12 -> 8
Other:
- title: WM8978 Codec -> WM8978 Codec and Microphone Front End
