File: pcb/WM8978.kicad_pcb (KiCad board)
At the start: 2 copper layers, 39.5 x 74.8 mm, 54 parts, among them CN2 HEADPHONE 3.5mm, J2 JLINK SWD, U1 ATSAMD21E18A-A, U15 TLV1117LV33DCYR, U16 WM8978CGEFL/RV, U17 TPS2553DBVR, Y1 12MHz / 3.3V / 50ppm, Y2 12.288MHz / 3.3V / 50ppm

Commit message: 保留最新 PCB 布局存档并更新模型检查记录
纳入 02:13 存档中的 R71 位置、供电及 SWCLK 走线调整，保留所有原始模型绑定。
更新几何、DRC、STEP 对齐验证与 3D 预览；未连接项和原理图一致性问题均为零，DRC 类型及数量不变。
Parts:
- moved R71 1.50 mm to (124.8, 85.2)
Routing:
- net +3V3: track 249.3 -> 247.8 mm
Changed lines of the file:
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@@
 	(footprint "Resistor_SMD:R_0603_1608Metric"
 		(layer "F.Cu")
-		(at 123.25 85.2 -90)
+		(at 124.75 85.2 -90)
 		(descr "Resistor SMD 0603 (1608 Metric), square (rectangular) end terminal, IPC-7351 nominal, (Body size source: IPC-SM-782 page 72, https://www.pcb-3d.com/wordpress/wp-content/uploads/ipc-sm-782a_amendment_1_and_2.pdf)")
 		(tags "resistor")
@@
 	)
 	(segment
+		(start 124.775 84.4)
+		(end 124.75 84.375)
+		(width 0.4)
+		(layer "F.Cu")
+		(net "+3V3")
+	)
+	(segment
 		(start 132.452472 86)
 		(end 130.5 87.952472)
@@
 	)
 	(segment
+		(start 131.0875 84.4)
+		(end 124.775 84.4)
+		(width 0.4)
+		(layer "F.Cu")
+		(net "+3V3")
+	)
+	(segment
 		(start 153.5 79)
 		(end 152.01384 80.48616)
@@
 	)
 	(segment
-		(start 131.0875 84.4)
-		(end 123.275 84.4)
-		(width 0.4)
-		(layer "F.Cu")
-		(net "+3V3")
-	)
-	(segment
 		(start 118.225 90.45)
 		(end 125.45 90.45)
@@
 	)
 	(segment
-		(start 124.075 85.2)
-		(end 131.0875 85.2)
+		(start 124.75 86.025)
+		(end 125.575 85.2)
 		(width 0.2)
 		(layer "F.Cu")
@@
 	)
 	(segment
-		(start 118.225 85.45)
-		(end 122.675 85.45)
+		(start 124.75 86.025)
+		(end 124.75 85.95)
 		(width 0.2)
 		(layer "F.Cu")
@@
 	)
 	(segment
-		(start 123.25 86.025)
-		(end 124.075 85.2)
+		(start 124.75 85.95)
+		(end 124.25 85.45)
 		(width 0.2)
 		(layer "F.Cu")
@@
 	)
 	(segment
-		(start 122.675 85.45)
-		(end 123.25 86.025)
+		(start 118.225 85.45)
+		(end 124.25 85.45)
+		(width 0.2)
+		(layer "F.Cu")
+		(net "/SWCLK")
+	)
+	(segment
+		(start 125.575 85.2)
+		(end 131.0875 85.2)
 		(width 0.2)
 		(layer "F.Cu")
